File: sra_board.kicad_sch (KiCad schematic)
At the start: 162 parts, among them J1 Conn_01x14_Pin, J10 Conn_01x03_Pin, J11 Conn_01x03_Pin, J12 Conn_01x03_Pin, J13 MPU0650, J14 LSA, J15 OLED, J16 Conn_01x03_Pin, J17 Conn_01x03_Pin, J18 Conn_01x03_Pin, J3 Conn_01x08_Pin, J4 Conn_01x14_Pin, J5 USB_C_Receptacle_USB2.0_16P, J6 B2B-XH-A_LF__SN_, J7 B2B-XH-A_LF__SN_, J8 B2B-XH-A_LF__SN_, J9 Conn_01x03_Pin, Q1 SS8050, Q2 SS8050, Q3 AO3400A, Q4 AO3401A, Q5 AO3401A, Q6 AO3401A, Q7 AO3401A, SW1 SW_0, SW2 SW_EN, SW3 Switch, SW4 Switch, SW5 SW_Wuerth_450301014042, SW6 SW_Wuerth_450301014042, U1 MAX7219CWG_T, U2 CH340C, U3 TB6612FNG H-bridge Motor Driv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, U5 CN3303, U6 TPS562202, U7 ME6211C33M5, U8 ESP32-WROOM-32E

Commit message: Finishing the routing
Parts:
- C19: footprint Capacitor_SMD:C_0603_1608Metric -> Capacitor_SMD:C_0805_2012Metric
- J14: footprint Connector_PinSocket_2.54mm:PinSocket_1x08_P2.54mm_Vertical -> Connector_PinSocket_2.54mm:PinSocket_1x07_P2.54mm_Vertical
- J3: footprint Connector_PinHeader_2.54mm:PinHeader_1x09_P2.54mm_Vertical -> Connector_PinHeader_2.54mm:PinHeader_1x10_P2.54mm_Vertical; symbol Connector:Conn_01x09_Pin -> Connector:Conn_01x10_Pin
- JP1, JP2, JP3, JP4, JP5: footprint Jumper:SolderJumper-2_P1.3mm_Open_RoundedPad1.0x1.5mm -> Connector_PinHeader_2.54mm:PinHeader_1x02_P2.54mm_Vertical
- R13: footprint Resistor_SMD:R_0805_2012Metric -> Resistor_SMD:R_1206_3216Metric
Connections:
- net CLK is gone; now on net 18: J4.8 (Pin_8)
- net CS is gone; now on net 5: J4.9 (Pin_9)
- net Din is gone; now on net 23: J4.2 (Pin_2)
- net 0: now also J3.10 (Pin_10); no longer J3.9 (Pin_9)
- net 15: now also J3.6 (Pin_6)
- net 16: now also J3.8 (Pin_8); no longer J3.7 (Pin_7)
- net 2: now also J3.7 (Pin_7); no longer J3.6 (Pin_6)
- net 4: now also J3.9 (Pin_9); no longer J3.8 (Pin_8)
- net 7V4_Switch renamed 12V_Switch
- net 7v4 renamed 12V
Changed lines of the file:
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@@
 		)
 	)
-	(label "7v4"
+	(label "12V"
 		(at 387.096 87.376 0)
 		(effects
@@
 	)
 	(label "16"
-		(at 161.544 99.822 0)
+		(at 161.544 102.362 0)
 		(effects
 			(font
@@
 	)
 	(label "4"
-		(at 161.544 102.362 0)
+		(at 161.544 104.902 0)
 		(effects
 			(font
@@
 		)
 	)
-	(label "CLK"
+	(label "18"
 		(at 177.292 101.092 0)
 		(effects
@@
 		)
 	)
-	(label "7V4_Switch"
+	(label "12V_Switch"
 		(at 387.096 65.278 180)
 		(effects
@@
 		)
 	)
-	(label "7v4"
+	(label "12V"
 		(at 401.4216 43.4594 0)
 		(effects
@@
 		)
 	)
-	(label "7v4"
+	(label "12V"
 		(at 148.59 121.412 0)
 		(effects
@@
 		)
 	)
-	(label "Din"
+	(label "23"
 		(at 177.292 85.852 0)
 		(effects
@@
 	)
 	(label "0"
-		(at 161.544 104.902 0)
+		(at 161.544 107.442 0)
 		(effects
 			(font
@@
 		)
 	)
-	(label "7v4"
+	(label "12V"
 		(at 189.738 152.908 180)
 		(effects
@@
 		)
 	)
-	(label "CS"
+	(label "5"
 		(at 177.292 103.632 0)
 		(effects
@@
 	)
 	(label "2"
-		(at 161.544 97.282 0)
+		(at 161.544 99.822 0)
 		(effects
 			(font
@@
 		)
 	)
-	(label "7V4_Switch"
+	(label "12V_Switch"
 		(at 375.666 42.164 180)
 		(effects
@@
 		)
 	)
+	(label "15"
+		(at 161.544 97.282 0)
+		(effects
+			(font
+				(size 1.27 1.27)
+			)
+			(justify left bottom)
+		)
+	)
 	(label "33"
 		(at 150.114 104.902 0)
@@
 	)
 	(symbol
-		(lib_id "Connector:Conn_01x09_Pin")
+		(lib_id "Connector:Conn_01x10_Pin")
 		(at 156.464 94.742 0)
 		(unit 1)
@@
 			)
 		)
-		(property "Footprint" "Connector_PinHeader_2.54mm:PinHeader_1x09_P2.54mm_Vertical"
+		(property "Footprint" "Connector_PinHeader_2.54mm:PinHeader_1x10_P2.54mm_Vertical"
 			(at 156.464 94.742 0)
 			(hide yes)
@@
 			)
 		)
-		(property "Description" "Generic connector, single row, 01x09, script generated"
+		(property "Description" "Generic connector, single row, 01x10, script generated"
 			(at 156.464 94.742 0)
 			(hide yes)
@@
 		(pin "9"
 		)
+		(pin "10"
+		)
 		(instances
 			(project "sra_board"
@@
 			)
 		)
-		(property "Footprint" "Capacitor_SMD:C_0603_1608Metric"
+		(property "Footprint" "Capacitor_SMD:C_0805_2012Metric"
 			(at 24.4348 40.64 0)
 			(hide yes)
@@
 			)
 		)
-		(property "Footprint" "Jumper:SolderJumper-2_P1.3mm_Open_RoundedPad1.0x1.5mm"
+		(property "Footprint" "Connector_PinHeader_2.54mm:PinHeader_1x02_P2.54mm_Vertical"
 			(at 392.684 96.266 0)
 			(hide yes)
@@
 			)
 		)
-		(property "Footprint" "Jumper:SolderJumper-2_P1.3mm_Open_RoundedPad1.0x1.5mm"
+		(property "Footprint" "Connector_PinHeader_2.54mm:PinHeader_1x02_P2.54mm_Vertical"
 			(at 380.238 45.974 0)
 			(hide yes)
@@
 			)
 		)
-		(property "Footprint" "Jumper:SolderJumper-2_P1.3mm_Open_RoundedPad1.0x1.5mm"
+		(property "Footprint" "Connector_PinHeader_2.54mm:PinHeader_1x02_P2.54mm_Vertical"
 			(at 387.096 69.85 0)
 			(hide yes)
@@
 			)
 		)
-		(property "Footprint" "Resistor_SMD:R_0805_2012Metric"
+		(property "Footprint" "Resistor_SMD:R_1206_3216Metric"
 			(at 66.294 128.27 90)
 			(hide yes)
@@
 			)
 		)
-		(property "Footprint" "Connector_PinSocket_2.54mm:PinSocket_1x08_P2.54mm_Vertical"
+		(property "Footprint" "Connector_PinSocket_2.54mm:PinSocket_1x07_P2.54mm_Vertical"
 			(at 276.86 130.048 0)
 			(hide yes)
@@
 			)
 		)
-		(property "Footprint" "Jumper:SolderJumper-2_P1.3mm_Open_RoundedPad1.0x1.5mm"
+		(property "Footprint" "Connector_PinHeader_2.54mm:PinHeader_1x02_P2.54mm_Vertical"
 			(at 177.546 161.036 0)
 			(hide yes)
@@
 			)
 		)
-		(property "Footprint" "Jumper:SolderJumper-2_P1.3mm_Open_RoundedPad1.0x1.5mm"
+		(property "Footprint" "Connector_PinHeader_2.54mm:PinHeader_1x02_P2.54mm_Vertical"
 			(at 379.73 25.908 0)
 			(hide yes)
