File: sra_board.kicad_sch (KiCad schematic)
At the start: 168 parts, among them J10 Conn_01x03_Pin, J11 Conn_01x08_Pin, J12 Conn_01x07_Pin, J13 Conn_01x04_Pin, J14 Conn_01x02_Pin, J15 Conn_01x02_Pin, J16 Conn_01x02_Pin, J17 USB_C_Receptacle_USB2.0_16P, J18 Conn_01x10_Pin, J19 Conn_01x10_Pin, J20 Conn_01x10_Pin, J3 Conn_01x03_Pin, J5 Conn_01x03_Pin, J6 Conn_01x03_Pin, J7 Conn_01x03_Pin, J8 Conn_01x03_Pin, J9 Conn_01x03_Pin, Q1 SS8050, Q2 SS8050, Q3 AO4435, Q4 AO4468, SW3 SW_IO0, SW4 Switch, SW5 SW_EN, SW6 Switch, U1 MAX7219CWG_T, U2 ESP32-WROOM-32E, U3 TPS562200, U4 ME6211C33M5, U5 CH340C, U7 CN3303, U8 TB6612FNG H-bridge Motor Driv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

Commit message: Done Silkscreen
Parts:
- removed H2, H4: MountingHole, MountingHole:MountingHole_3.2mm_M3, symbol Mechanical:MountingHole
- C12, C13, C14, C17, C18, C21, C22, C23, C24: footprint Capacitor_SMD:C_0603_1608Metric -> Capacitor_SMD:C_1206_3216Metric
Changed lines of the file:
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@@
 			)
 		)
-		(property "Footprint" "Capacitor_SMD:C_0603_1608Metric"
+		(property "Footprint" "Capacitor_SMD:C_1206_3216Metric"
 			(at 180.8988 179.07 0)
 			(hide yes)
@@
 			)
 		)
-		(property "Footprint" "Capacitor_SMD:C_0603_1608Metric"
+		(property "Footprint" "Capacitor_SMD:C_1206_3216Metric"
 			(at 88.646 162.7632 0)
 			(hide yes)
@@
 	)
 	(symbol
-		(lib_id "Mechanical:MountingHole")
-		(at 367.284 126.746 0)
-		(unit 1)
-		(body_style 1)
-		(exclude_from_sim no)
-		(in_bom no)
-		(on_board yes)
-		(in_pos_files yes)
-		(dnp no)
-		(fields_autoplaced yes)
-		(property "Reference" "H2"
-			(at 370.586 125.4759 0)
-			(show_name no)
-			(do_not_autoplace no)
-			(effects
-				(font
-					(size 1.27 1.27)
-				)
-				(justify left)
-			)
-		)
-		(property "Value" "MountingHole"
-			(at 370.586 128.0159 0)
-			(show_name no)
-			(do_not_autoplace no)
-			(effects
-				(font
-					(size 1.27 1.27)
-				)
-				(justify left)
-			)
-		)
-		(property "Footprint" "MountingHole:MountingHole_3.2mm_M3"
-			(at 367.284 126.746 0)
-			(hide yes)
-			(show_name no)
-			(do_not_autoplace no)
-			(effects
-				(font
-					(size 1.27 1.27)
-				)
-			)
-		)
-		(property "Datasheet" ""
-			(at 367.284 126.746 0)
-			(hide yes)
-			(show_name no)
-			(do_not_autoplace no)
-			(effects
-				(font
-					(size 1.27 1.27)
-				)
-			)
-		)
-		(property "Description" "Mounting Hole without connection"
-			(at 367.284 126.746 0)
-			(hide yes)
-			(show_name no)
-			(do_not_autoplace no)
-			(effects
-				(font
-					(size 1.27 1.27)
-				)
-			)
-		)
-		(instances
-			(project "sra_board"
-				(path "/294e2e5f-a7b9-4d81-904c-b55cda9b730c"
-					(reference "H2")
-					(unit 1)
-				)
-			)
-		)
-	)
-	(symbol
 		(lib_id "Device:C")
 		(at 34.036 163.068 0)
@@
 			)
 		)
-		(property "Footprint" "Capacitor_SMD:C_0603_1608Metric"
+		(property "Footprint" "Capacitor_SMD:C_1206_3216Metric"
 			(at 35.0012 166.878 0)
 			(hide yes)
@@
 			)
 		)
-		(property "Footprint" "Capacitor_SMD:C_0603_1608Metric"
+		(property "Footprint" "Capacitor_SMD:C_1206_3216Metric"
 			(at 28.6512 166.878 0)
 			(hide yes)
@@
 			)
 		)
-		(property "Footprint" "Capacitor_SMD:C_0603_1608Metric"
+		(property "Footprint" "Capacitor_SMD:C_1206_3216Metric"
 			(at 190.9572 153.67 0)
 			(hide yes)
@@
 			)
 		)
-		(property "Footprint" "Capacitor_SMD:C_0603_1608Metric"
+		(property "Footprint" "Capacitor_SMD:C_1206_3216Metric"
 			(at 88.646 169.1132 0)
 			(hide yes)
@@
 			)
 		)
-		(property "Footprint" "Capacitor_SMD:C_0603_1608Metric"
+		(property "Footprint" "Capacitor_SMD:C_1206_3216Metric"
 			(at 175.3108 179.07 0)
 			(hide yes)
@@
 	)
 	(symbol
-		(lib_id "Mechanical:MountingHole")
-		(at 388.62 126.492 0)
-		(unit 1)
-		(body_style 1)
-		(exclude_from_sim no)
-		(in_bom no)
-		(on_board yes)
-		(in_pos_files yes)
-		(dnp no)
-		(fields_autoplaced yes)
-		(property "Reference" "H4"
-			(at 391.922 125.2219 0)
-			(show_name no)
-			(do_not_autoplace no)
-			(effects
-				(font
-					(size 1.27 1.27)
-				)
-				(justify left)
-			)
-		)
-		(property "Value" "MountingHole"
-			(at 391.922 127.7619 0)
-			(show_name no)
-			(do_not_autoplace no)
-			(effects
-				(font
-					(size 1.27 1.27)
-				)
-				(justify left)
-			)
-		)
-		(property "Footprint" "MountingHole:MountingHole_3.2mm_M3"
-			(at 388.62 126.492 0)
-			(hide yes)
-			(show_name no)
-			(do_not_autoplace no)
-			(effects
-				(font
-					(size 1.27 1.27)
-				)
-			)
-		)
-		(property "Datasheet" ""
-			(at 388.62 126.492 0)
-			(hide yes)
-			(show_name no)
-			(do_not_autoplace no)
-			(effects
-				(font
-					(size 1.27 1.27)
-				)
-			)
-		)
-		(property "Description" "Mounting Hole without connection"
-			(at 388.62 126.492 0)
-			(hide yes)
-			(show_name no)
-			(do_not_autoplace no)
-			(effects
-				(font
-					(size 1.27 1.27)
-				)
-			)
-		)
-		(instances
-			(project "sra_board"
-				(path "/294e2e5f-a7b9-4d81-904c-b55cda9b730c"
-					(reference "H4")
-					(unit 1)
-				)
-			)
-		)
-	)
-	(symbol
 		(lib_id "MMBT8050:MMBT8050")
 		(at 191.262 129.032 0)
@@
 			)
 		)
-		(property "Footprint" "Capacitor_SMD:C_0603_1608Metric"
+		(property "Footprint" "Capacitor_SMD:C_1206_3216Metric"
 			(at 41.3512 166.878 0)
 			(hide yes)
@@
 			)
 		)
-		(property "Footprint" "Capacitor_SMD:C_0603_1608Metric"
+		(property "Footprint" "Capacitor_SMD:C_1206_3216Metric"
 			(at 185.3692 153.67 0)
 			(hide yes)

Commit message: Done Silkscreen
Parts:
- removed J12: Conn_01x07_Pin, Connector_JST:JST_EH_S7B-EH_1x07_P2.50mm_Horizontal, symbol Connector:Conn_01x07_Pin
- added J1: Conn_01x08_Pin, Connector_FFC-FPC:JUSHUO_AFA07-S08FCA-00_1x8-1MP_P1.0mm_Horizontal, symbol Connector:Conn_01x08_Pin
- added R16: 0, Resistor_SMD:R_0603_1608Metric, symbol Device:R
- C12, C13, C14, C17, C18: footprint Capacitor_SMD:C_1206_3216Metric -> Capacitor_SMD:C_0603_1608Metric
- C21, C23: value 22uf -> NC; footprint Capacitor_SMD:C_1206_3216Metric -> Capacitor_SMD:C_0603_1608Metric
- J16: footprint Connector_JST:JST_VH_B2PS-VH_1x02_P3.96mm_Horizontal -> Connector_BarrelJack:BarrelJack_Wuerth_6941xx301002
- L1: value 3.3uH -> 4.7uH
- R14: value 20m -> 40m
- SW6: footprint Button_Switch_THT:SW_Push_2P2T_Toggle_CK_PVA2OAH5xxxxxxV2 -> Button_Switch_SMD:SW_SPDT_PCM12
- U7: MANUFACTURER (none) -> CONSONANCE(上海如韵); Manufacturer CONSONANCE(上海如韵) -> (none)
Connections:
- net 12V: now also R16.2
- net 32: now also J1.8 (Pin_8)
- net 34: now also J1.6 (Pin_6)
- net 35: now also J1.7 (Pin_7)
- net 36: now also J1.4 (Pin_4)
- net 39: now also J1.5 (Pin_5)
- net 3V3: now also J1.2 (Pin_2)
- net BAT: now also R16.1
- net GND: now also J1.3 (Pin_3)
- no-connect marks 15 -> 16
Other:
- note added: "CN3303 ICH = 1A (Charging IC)"
- note removed: "CN3303 (Charging IC)"
