File: sra_board.kicad_sch (KiCad schematic)
At the start: 148 parts, among them J1 Barrel_Jack, J10 B2B-XH-A_LF__SN_, J11 Conn_01x03_Pin, J12 Conn_01x03_Pin, J13 Conn_01x03_Pin, J14 MPU0650, J15 Conn_01x03_Pin, J16 LSA, J17 OLED, J18 B2B-XH-A_LF__SN_, J2 Conn_01x03_Pin, J3 USB_C_Receptacle_USB2.0_16P, J4 Conn_01x14_Pin, J5 Conn_01x03_Pin, J6 Conn_01x08_Pin, J7 Conn_01x03_Pin, J8 Conn_01x14_Pin, J9 B2B-XH-A_LF__SN_, Q3 SS8050, Q4 SS8050, Q7 ZXMP4A16GTA, SW1 SW_0, SW2 SW_EN, SW3 SW_Wuerth_450301014042, SW4 SW_Wuerth_450301014042, U1 ESP32-WROOM-32E, U3 CH340C, U4 TB6612FNG H-bridge Motor Driv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, U5 AMS1117-3.3, U6 MAX7219CWG_T, U7 TPS54302

Commit message: Making minor fixes in pcb
Parts:
- H1, H2, H3, H4: footprint MountingHole:MountingHole_3.2mm_M3_DIN965 -> MountingHole:MountingHole_3.2mm_M3_DIN965_Pad
Connections:
- net 12V: now also R25.2; no longer D75.2 (A)
- net 5V_P: now also R24.2; no longer D74.2 (A)
- net GND: now also D74.1 (K), D75.1 (K); no longer R24.1, R25.1
- new net: D75.2 (A), R25.1
- new net: D74.2 (A), R24.1
Other:
- moved on the sheet: D74, D75, R24, R25
Changed lines of the file:
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@@
 	)
 	(junction
+		(at 362.204 168.402)
+		(diameter 0)
+		(color 0 0 0 0)
+	)
+	(junction
 		(at 211.328 60.706)
 		(diameter 0)
@@
 	)
 	(junction
+		(at 359.664 60.452)
+		(diameter 0)
+		(color 0 0 0 0)
+	)
+	(junction
 		(at 152.654 31.242)
 		(diameter 0)
@@
 	)
 	(junction
-		(at 362.204 168.402)
-		(diameter 0)
-		(color 0 0 0 0)
-	)
-	(junction
 		(at 315.976 93.726)
 		(diameter 0)
@@
 	)
 	(junction
-		(at 359.664 60.452)
-		(diameter 0)
-		(color 0 0 0 0)
-	)
-	(junction
 		(at 224.536 53.086)
 		(diameter 0)
@@
 	(wire
 		(pts
+			(xy 362.204 168.402) (xy 359.918 168.402)
+		)
+		(stroke
+			(width 0)
+			(type default)
+		)
+	)
+	(wire
+		(pts
 			(xy 216.154 123.698) (xy 218.186 123.698)
 		)
@@
 	(wire
 		(pts
-			(xy 359.664 60.452) (xy 359.664 70.104)
+			(xy 359.664 54.864) (xy 359.664 60.452)
 		)
 		(stroke
@@
 	(wire
 		(pts
-			(xy 363.728 168.402) (xy 359.918 168.402)
+			(xy 363.728 168.402) (xy 362.204 168.402)
 		)
 		(stroke
@@
 	(wire
 		(pts
+			(xy 359.664 60.452) (xy 359.664 70.104)
+		)
+		(stroke
+			(width 0)
+			(type default)
+		)
+	)
+	(wire
+		(pts
 			(xy 247.396 73.406) (xy 247.396 83.566)
 		)
@@
 	(wire
 		(pts
-			(xy 359.664 54.864) (xy 359.664 60.452)
-		)
-		(stroke
-			(width 0)
-			(type default)
-		)
-	)
-	(wire
-		(pts
 			(xy 188.722 17.272) (xy 188.722 21.082)
 		)
@@
 			)
 		)
-		(property "Footprint" "MountingHole:MountingHole_3.2mm_M3_DIN965"
+		(property "Footprint" "MountingHole:MountingHole_3.2mm_M3_DIN965_Pad"
 			(at 365.506 144.018 0)
 			(hide yes)
@@
 	(symbol
 		(lib_id "Device:R_Small")
-		(at 368.046 60.452 270)
+		(at 362.204 60.452 270)
 		(mirror x)
 		(unit 1)
@@
 		(dnp no)
 		(property "Reference" "R25"
-			(at 367.03 56.134 0)
+			(at 361.188 56.134 0)
 			(show_name no)
 			(do_not_autoplace no)
@@
 		)
 		(property "Value" "330"
-			(at 369.062 55.118 0)
+			(at 363.22 55.118 0)
 			(show_name no)
 			(do_not_autoplace no)
@@
 		)
 		(property "Footprint" "Resistor_SMD:R_0805_2012Metric"
-			(at 368.046 60.452 0)
+			(at 362.204 60.452 0)
 			(hide yes)
 			(show_name no)
@@
 		)
 		(property "Datasheet" ""
-			(at 368.046 60.452 0)
+			(at 362.204 60.452 0)
 			(hide yes)
 			(show_name no)
@@
 		)
 		(property "Description" "Resistor, small symbol"
-			(at 368.046 60.452 0)
+			(at 362.204 60.452 0)
 			(hide yes)
 			(show_name no)
@@
 	(symbol
 		(lib_id "Device:R_Small")
-		(at 362.204 176.784 180)
+		(at 362.204 170.942 180)
 		(unit 1)
 		(body_style 1)
@@
 		(dnp no)
 		(property "Reference" "R24"
-			(at 363.474 175.26 0)
+			(at 363.474 169.418 0)
 			(show_name no)
 			(do_not_autoplace no)
@@
 		)
 		(property "Value" "330"
-			(at 363.22 177.292 0)
+			(at 363.22 171.45 0)
 			(show_name no)
 			(do_not_autoplace no)
@@
 		)
 		(property "Footprint" "Resistor_SMD:R_0805_2012Metric"
-			(at 362.204 176.784 0)
+			(at 362.204 170.942 0)
 			(hide yes)
 			(show_name no)
@@
 		)
 		(property "Datasheet" ""
-			(at 362.204 176.784 0)
+			(at 362.204 170.942 0)
 			(hide yes)
 			(show_name no)
@@
 		)
 		(property "Description" "Resistor, small symbol"
-			(at 362.204 176.784 0)
+			(at 362.204 170.942 0)
 			(hide yes)
 			(show_name no)
@@
 			)
 		)
-		(property "Footprint" "MountingHole:MountingHole_3.2mm_M3_DIN965"
+		(property "Footprint" "MountingHole:MountingHole_3.2mm_M3_DIN965_Pad"
 			(at 364.744 128.27 0)
 			(hide yes)
@@
 			)
 		)
-		(property "Footprint" "MountingHole:MountingHole_3.2mm_M3_DIN965"
+		(property "Footprint" "MountingHole:MountingHole_3.2mm_M3_DIN965_Pad"
 			(at 343.662 128.27 0)
 			(hide yes)
@@
 			)
 		)
-		(property "Footprint" "MountingHole:MountingHole_3.2mm_M3_DIN965"
+		(property "Footprint" "MountingHole:MountingHole_3.2mm_M3_DIN965_Pad"
 			(at 344.17 143.764 0)
 			(hide yes)
@@
 	(symbol
 		(lib_id "Device:LED_Small")
-		(at 362.204 60.452 0)
+		(at 368.046 60.452 0)
 		(mirror y)
 		(unit 1)
@@
 		(dnp no)
 		(property "Reference" "D75"
-			(at 361.188 57.912 90)
+			(at 367.03 57.912 90)
 			(show_name no)
 			(do_not_autoplace no)
@@
 		)
 		(property "Value" "LED"
-			(at 363.474 57.15 90)
+			(at 369.316 57.15 90)
 			(show_name no)
 			(do_not_autoplace no)
@@
 		)
 		(property "Footprint" "LED_SMD:LED_0805_2012Metric"
-			(at 362.204 60.452 90)
+			(at 368.046 60.452 90)
 			(hide yes)
 			(show_name no)
@@
 		)
 		(property "Datasheet" ""
-			(at 362.204 60.452 90)
+			(at 368.046 60.452 90)
 			(hide yes)
 			(show_name no)
@@
 		)
 		(property "Description" "Light emitting diode, small symbol"
-			(at 362.204 60.452 0)
+			(at 368.046 60.452 0)
 			(hide yes)
 			(show_name no)
@@
 		)
 		(property "Sim.Pin" "1=K 2=A"
-			(at 362.204 60.452 0)
+			(at 368.046 60.452 0)
 			(hide yes)
 			(show_name no)
@@
 	(symbol
 		(lib_id "Device:LED_Small")
-		(at 362.204 170.942 90)
+		(at 362.204 176.784 90)
 		(unit 1)
 		(body_style 1)
@@
 		(dnp no)
 		(property "Reference" "D74"
-			(at 359.664 169.926 90)
+			(at 359.664 175.768 90)
 			(show_name no)
 			(do_not_autoplace no)
@@
 		)
 		(property "Value" "LED"
-			(at 358.902 172.212 90)
+			(at 358.902 178.054 90)
 			(show_name no)
 			(do_not_autoplace no)
@@
 		)
 		(property "Footprint" "LED_SMD:LED_0805_2012Metric"
-			(at 362.204 170.942 90)
+			(at 362.204 176.784 90)
 			(hide yes)
 			(show_name no)
@@
 		)
 		(property "Datasheet" ""
-			(at 362.204 170.942 90)
+			(at 362.204 176.784 90)
 			(hide yes)
 			(show_name no)
@@
 		)
 		(property "Description" "Light emitting diode, small symbol"
-			(at 362.204 170.942 0)
+			(at 362.204 176.784 0)
 			(hide yes)
 			(show_name no)
@@
 		)
 		(property "Sim.Pin" "1=K 2=A"
-			(at 362.204 170.942 0)
+			(at 362.204 176.784 0)
 			(hide yes)
 			(show_name no)
