File: sra_board.kicad_pcb (KiCad board)
At the start: 2 copper layers, 97.6 x 65.8 mm, 165 parts, among them J10 Conn_01x03_Pin, J11 Conn_01x08_Pin, J12 Conn_01x07_Pin, J13 Conn_01x04_Pin, J14 Conn_01x02_Pin, J15 Conn_01x02_Pin, J16 Conn_01x02_Pin, J17 USB_C_Receptacle_USB2.0_16P, J18 Conn_01x10_Pin, J19 Conn_01x10_Pin, J20 Conn_01x10_Pin, J3 Conn_01x03_Pin, J5 Conn_01x03_Pin, J6 Conn_01x03_Pin, J7 Conn_01x03_Pin, J8 Conn_01x03_Pin, J9 Conn_01x03_Pin, Q1 SS8050, Q2 SS8050, Q3 AO4435, Q4 AO4468, SW3 SW_IO0, SW4 Switch, SW5 SW_EN, SW6 Switch, U2 ESP32-WROOM-32E, U4 ME6211C33M5, U5 CH340C, U6 TPS562202, U8 TB6612FNG H-bridge Motor Driv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

Commit message: Added something
Parts:
- added L1: 3.3uH, Inductor_SMD:L_TDK_VLS6045EX_VLS6045AF, F.Cu at (113.4, 93.4)
- added U1: MAX7219CWG_T, max:SOIC24, F.Cu at (128.5, 71.9)
- added U7: CN3303, CN3303N:SOP-8_L4.9-W3.9-P1.27-LS6.0-BL, F.Cu at (114.8, 111.2)
- D73: footprint Diode_SMD:D_SMB -> Diode_SMD:D_SMA
- F1, F2: footprint Fuse:Fuse_Littelfuse-LVR100 -> Fuse:Fuse_1812_4532Metric
- H1, H2, H3, H4, H5, H6: footprint MountingHole:MountingHole_3.2mm_M3 -> MountingHole:MountingHole_3.2mm_M3_Pad_Via
- J16: footprint Connector_JST:JST_EH_S2B-EH_1x02_P2.50mm_Horizontal -> Connector_JST:JST_VH_B2PS-VH_1x02_P3.96mm_Horizontal
- moved L2 85.4 mm to (111.8, 127.5)
- moved H1 68.2 mm to (24.6, 162.5)
- moved H2 68.2 mm to (24.6, 170.5)
- moved H3 68.2 mm to (32.5, 162.5)
- moved H4 68.2 mm to (32.5, 170.5)
- moved H5 68.2 mm to (40.5, 162.5)
- moved H6 68.2 mm to (40.5, 170.5)
- moved Q3 54.4 mm to (110.1, 99.7)
- moved D1 54.2 mm to (100.5, 220.2)
- moved D69 51.7 mm to (128.7, 103.3)
- moved D72 49.6 mm to (128.7, 114.5)
- moved Q1 49.5 mm to (81.1, 144.5)
- moved D71 49.5 mm to (128.5, 110.0)
- moved D37 47.0 mm to (77.3, 137.8)
- moved Q4 46.2 mm to (117.4, 99.8)
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Other:
- board size 97.6 x 65.8 mm -> 90 x 94.1 mm

Commit message: Made some arrengements
Parts:
- moved D1 131.6 mm to (82.2, 89.8), turned to 180 degrees
- moved D57 119.3 mm to (106.6, 89.9)
- moved D59 119.3 mm to (106.6, 95.1)
- moved D60 119.3 mm to (106.6, 97.7)
- moved D58 119.3 mm to (106.6, 92.5)
- moved D33 118.9 mm to (96.5, 89.9)
- moved D34 118.9 mm to (96.5, 92.5)
- moved D35 118.9 mm to (96.5, 95.1)
- moved D36 118.9 mm to (96.5, 97.7)
- moved D9 118.6 mm to (85.8, 89.8)
- moved D11 118.6 mm to (85.8, 95.0)
- moved D12 118.6 mm to (85.8, 97.5)
- moved D10 118.6 mm to (85.8, 92.4)
- moved D24 109.0 mm to (89.5, 107.2)
- moved D43 108.7 mm to (99.9, 95.0)
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Other:
- board size 90 x 94.1 mm -> 218.2 x 121.8 mm

Commit message: Made some placements
Parts:
- added J1: Conn_01x03_Pin, Connector_PinHeader_2.54mm:PinHeader_1x03_P2.54mm_Vertical, F.Cu at (116.8, 114.3)
- moved D8 80.9 mm to (146.5, 57.8), turned to -135 degrees
- moved D7 77.7 mm to (143.9, 57.8), turned to -135 degrees
- moved J10 76.7 mm to (13.8, 142.0)
- moved J7 76.7 mm to (17.9, 141.8)
- moved J8 76.7 mm to (21.9, 141.6)
- moved J9 76.7 mm to (25.8, 141.6)
- moved D16 76.6 mm to (146.5, 60.4), turned to -135 degrees
- moved D6 74.1 mm to (141.4, 57.8), turned to -135 degrees
- moved D15 73.1 mm to (144.0, 60.4), turned to -135 degrees
- moved D24 72.2 mm to (146.5, 62.9), turned to -135 degrees
- moved U1 70.7 mm to (141.2, 23.0), turned to 90 degrees
- moved D5 70.6 mm to (139.0, 57.8), turned to -135 degrees
- moved D14 69.4 mm to (141.4, 60.4), turned to -135 degrees
- moved D23 68.9 mm to (143.9, 62.9), turned to -135 degrees
- moved D32 67.8 mm to (146.5, 65.5), turned to -135 degrees
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Other:
- board size 218.2 x 121.8 mm -> 106.9 x 106.5 mm

Commit message: Done some arrengements
Parts:
- removed J1: Conn_01x03_Pin, Connector_PinHeader_2.54mm:PinHeader_1x03_P2.54mm_Vertical
- moved U1 83.8 mm to (94.3, 92.5), turned to 180 degrees
- moved D13 64.1 mm to (95.9, 107.7)
- moved D21 64.1 mm to (95.9, 110.3)
- moved D29 64.1 mm to (95.9, 112.9)
- moved D37 64.1 mm to (95.9, 115.4)
- moved D45 64.1 mm to (95.9, 118.0)
- moved D5 64.1 mm to (95.9, 105.2)
- moved D53 64.1 mm to (95.9, 120.6)
- moved D61 64.1 mm to (95.9, 123.3)
- moved D1 64.1 mm to (85.9, 105.2)
- moved D10 64.1 mm to (88.4, 107.7)
- moved D11 64.1 mm to (90.9, 107.7)
- moved D12 64.1 mm to (93.4, 107.7)
- moved D14 64.1 mm to (98.2, 107.7)
- moved D15 64.1 mm to (100.9, 107.7)
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Other:
- board size 106.9 x 106.5 mm -> 106.6 x 92.7 mm

Commit message: Component Placement Done
Parts:
- added kibuzzard-6A672D04: G***, kibuzzard-6A672D04, F.Cu at (106.1, 60.3)
- added kibuzzard-6A672D28: G***, kibuzzard-6A672D28, F.Cu at (110.2, 60.3)
- added kibuzzard-6A672D33: G***, kibuzzard-6A672D33, F.Cu at (114.5, 60.3)
- added kibuzzard-6A672D4A: G***, kibuzzard-6A672D4A, F.Cu at (101.7, 60.3)
- added kibuzzard-6A672DD5: G***, kibuzzard-6A672DD5, F.Cu at (154.4, 60.3)
- added kibuzzard-6A672DEC: G***, kibuzzard-6A672DEC, F.Cu at (160.0, 60.3)
- added kibuzzard-6A673709: G***, kibuzzard-6A673709, F.Cu at (172.1, 79.2)
- added kibuzzard-6A6737F7: G***, kibuzzard-6A6737F7, F.Cu at (93.7, 88.7)
- added kibuzzard-6A67380D: G***, kibuzzard-6A67380D, F.Cu at (93.7, 93.1)
- added kibuzzard-6A67381F: G***, kibuzzard-6A67381F, F.Cu at (93.7, 97.4)
- added kibuzzard-6A673958: G***, kibuzzard-6A673958, F.Cu at (101.8, 113.9)
- added kibuzzard-6A673964: G***, kibuzzard-6A673964, F.Cu at (101.8, 103.4)
- added kibuzzard-6A673F05: G***, kibuzzard-6A673F05, F.Cu at (125.7, 112.3)
- added kibuzzard-6A674FE8: G***, kibuzzard-6A674FE8, F.Cu at (166.3, 91.3)
- added kibuzzard-6A675360: G***, kibuzzard-6A675360, F.Cu at (111.4, 114.8)
- added kibuzzard-6A675DE5: G***, kibuzzard-6A675DE5, F.Cu at (170.5, 110.7)
- added kibuzzard-6A6763A9: G***, kibuzzard-6A6763A9, F.Cu at (93.9, 71.3)
- H1, H3, H5, H6: footprint MountingHole:MountingHole_3.2mm_M3_Pad_Via -> MountingHole:MountingHole_3.2mm_M3_DIN965_Pad
- H2, H4: footprint MountingHole:MountingHole_3.2mm_M3_Pad_Via -> MountingHole:MountingHole_3.2mm_M3
- SW4: footprint Button_Switch_THT:SW_Push_2P2T_Toggle_CK_PVA2OAH5xxxxxxV2 -> Button_Switch_SMD:SW_SPDT_PCM12
- moved C10 222.1 mm to (152.3, 66.0), turned to 90 degrees
- moved C9 213.6 mm to (164.1, 80.8)
- moved C8 213.5 mm to (164.1, 78.5)
- moved C1 205.9 mm to (158.1, 66.0), turned to -90 degrees
- moved C11 205.8 mm to (162.0, 66.0), turned to 90 degrees
- moved R1 204.9 mm to (156.3, 66.0), turned to 90 degrees
- moved R11 204.7 mm to (160.0, 66.0), turned to -90 degrees
- moved C4 204.7 mm to (167.4, 81.6), turned to 90 degrees
- moved R12 204.1 mm to (154.3, 66.0), turned to -90 degrees
- moved C5 203.4 mm to (167.4, 85.7), turned to 90 degrees
- moved R22 201.6 mm to (164.1, 69.7), turned to 180 degrees
- moved R5 201.4 mm to (158.9, 81.8)
- moved R13 201.1 mm to (169.9, 81.6), turned to 90 degrees
- moved R18 198.2 mm to (161.3, 89.6), turned to 180 degrees
- moved R19 197.6 mm to (156.5, 89.8), turned to -90 degrees
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Connections:
- C2 pad 1: /5V -> /5V_P
- C3 pad 1: /5V -> /5V_P
- TP3 pad 1: /7v4 -> /12V
- U8 pad 1: /7v4 -> /12V
- U8 pad 2: /3V3 -> /12V
Routing:
- net /C5: track 0.00 -> 18.6 mm, vias 0 -> 8
- net /C3: track 0.00 -> 18.5 mm, vias 0 -> 9
- net /C1: track 0.00 -> 18.5 mm, vias 0 -> 8
- net /C4: track 0.00 -> 18.4 mm, vias 0 -> 8
- net /C2: track 0.00 -> 18.4 mm, vias 0 -> 8
- net /C8: track 0.00 -> 18.2 mm
- net /R4: track 0.00 -> 17.5 mm
- net /R8: track 0.00 -> 17.5 mm
- net /R7: track 0.00 -> 17.5 mm
- net /R6: track 0.00 -> 17.5 mm
- net /R5: track 0.00 -> 17.5 mm
- net /R3: track 0.00 -> 17.5 mm
- net /R2: track 0.00 -> 17.5 mm
- net /R1: track 0.00 -> 17.5 mm
- net /C7: track 0.00 -> 0.34 mm, vias 0 -> 8
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Other:
- board size 106.6 x 92.7 mm -> 81.1 x 66.3 mm
- board text added: "0"
- board text added: "0.1u"
- board text added: "10K"
- board text added: "10u"
- board text added: "12"
- board text added: "13"
- board text added: "14"
- board text added: "15"
- board text added: "16"
- board text added: "17"
- board text added: "18"
- board text added: "19"
- board text added: "1A"
- board text added: "1K"
- board text added: "1u"
- board text added: "2"
- board text added: "20m"
- board text added: "21"
- board text added: "22"
- board text added: "220"
- board text added: "22u"
- board text added: "23"
- board text added: "25"
- board text added: "26"
- board text added: "27"
- board text added: "32"
- board text added: "33"
- board text added: "330"
- board text added: "34"
- board text added: "35"
- board text added: "36"
- board text added: "39"
- board text added: "3V3"
- board text added: "4"
- board text added: "4.7K"
- board text added: "4.7uH"
- board text added: "5"
- board text added: "5.1K"
- board text added: "52K3"
- board text added: "5V"
- board text added: "680"
- board text added: "BAT"
- board text added: "CH340"
- board text added: "EN"
- board text added: "GND"
- board text added: "GREEN"
- board text added: "LDO"
- board text added: "NC"
- board text added: "Q1"
- board text added: "Q2"
- board text added: "Q3"
- board text added: "Q4"
- board text added: "RED"
- board text added: "RXD"
- board text added: "SCL"
- board text added: "SDA"
- board text added: "SS14"
- board text added: "SS34"
- board text added: "TXD"

Commit message: Done some routing
Parts:
- removed U6: TPS562202, Package_TO_SOT_SMD:SOT-563
- added U3: TPS562200, Package_TO_SOT_SMD:SOT-23-6, F.Cu at (149.9, 93.8)
- added kibuzzard-6A6A04C6: G***, kibuzzard-6A6A04C6, F.Cu at (157.9, 93.7)
- added kibuzzard-6A6A0879: G***, kibuzzard-6A6A0879, F.Cu at (105.3, 77.2)
- added kibuzzard-6A6A09BF: G***, kibuzzard-6A6A09BF, F.Cu at (111.6, 114.7)
- moved TP3 19.5 mm to (117.5, 111.5)
- moved kibuzzard-6A675360 9.10 mm to (120.5, 115.1), turned to 90 degrees
- moved C17 1.63 mm to (154.2, 98.9)
- moved R23 1.63 mm to (154.2, 100.7)
- moved C18 1.63 mm to (154.1, 96.9)
- moved R19 1.35 mm to (155.2, 89.6)
- moved C15 1.27 mm to (155.2, 93.7)
- moved C14 0.92 mm to (152.3, 89.6)
- moved L2 0.49 mm to (148.2, 98.9), turned to -90 degrees
- moved C13 0.49 mm to (149.4, 89.6)
- moved D74 0.25 mm to (162.4, 107.9)
- moved F1 0.25 mm to (161.2, 102.7)
- moved R50 0.25 mm to (160.1, 108.1)
- moved C12 0.16 mm to (146.6, 89.6)
- moved R17 0.12 mm to (153.2, 93.7)
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Routing:
- net /3V3: track 0.00 -> 244.9 mm, vias 0 -> 10
- net /5V_P: track 0.00 -> 161.2 mm, vias 0 -> 5
- net /22: track 0.00 -> 128.3 mm
- net /12V: track 0.00 -> 122.6 mm, vias 0 -> 6
- net /21: track 0.00 -> 116.7 mm
- net /39: track 0.00 -> 115.3 mm, vias 0 -> 1
- net /35: track 0.00 -> 108.6 mm, vias 0 -> 3
- net GND: track 0.00 -> 106.7 mm, vias 0 -> 27
- net /32: track 0.00 -> 102.5 mm, vias 0 -> 3
- net /25: track 0.00 -> 91.5 mm, vias 0 -> 2
- net /36: track 0.00 -> 90.0 mm, vias 0 -> 2
- net /18: track 0.00 -> 86.2 mm, vias 0 -> 1
- net /12: track 0.00 -> 84.8 mm, vias 0 -> 1
- net /5V_P_USB: track 0.00 -> 84.7 mm, vias 0 -> 3
- net /26: track 0.00 -> 84.2 mm, vias 0 -> 2
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- added copper zone on B.Cu, net GND
- added copper zone on F.Cu, net GND

Commit message: Done some more routing
Routing:
- net /C5: track 53.2 -> 42.3 mm
- net /R4: track 37.7 -> 36.5 mm
- net /C4: track 49.6 -> 48.4 mm
- net /34: track 75.9 -> 74.7 mm
- net /R8: track 41.2 -> 42.2 mm
- net /5: track 67.4 -> 68.4 mm
- net /R5: track 29.0 -> 28.1 mm
- net /5V_P: track 161.2 -> 160.3 mm

Commit message: Done Silkscreen
Parts:
- removed H2, H4: MountingHole, MountingHole:MountingHole_3.2mm_M3
- removed kibuzzard-6A6A0879: G***, kibuzzard-6A6A0879
- added G***: LOGO, logos:sra_skull_big, B.Cu at (105.9, 79.3)
- added G***: LOGO, logos:sra_logo_small_neg, B.Cu at (110.5, 115.2)
- added G***: LOGO, Logos:Lions_logo, B.Cu at (112.6, 94.6)
- added G***: LOGO, logos:espressif_logo, B.Cu at (134.4, 68.3)
- added H5: MountingHole, MountingHole:MountingHole_2.1mm, F.Cu at (98.2, 82.7)
- added H6: MountingHole, MountingHole:MountingHole_2.1mm, F.Cu at (113.2, 82.5)
- added J4: Barrel_Jack_Switch, Connector_BarrelJack:BarrelJack_Wuerth_6941xx301002, B.Cu at (162.4, 118.3)
- added kibuzzard-66914CE9: G***, kibuzzard-66914CE9, B.Cu at (134.4, 78.3)
- added kibuzzard-66921043: G***, kibuzzard-66921043, B.Cu at (134.4, 75.4)
- added kibuzzard-6A6CE0D4: G***, kibuzzard-6A6CE0D4, F.Cu at (122.5, 122.6)
- added kibuzzard-6A6CE942: G***, kibuzzard-6A6CE942, B.Cu at (133.8, 123.6)
- added kibuzzard-6A6CEA1C: G***, kibuzzard-6A6CEA1C, F.Cu at (105.5, 77.1)
- added kibuzzard-6A6CEC98: G***, kibuzzard-6A6CEC98, B.Cu at (157.1, 62.6)
- added kibuzzard-6A6CED08: G***, kibuzzard-6A6CED08, B.Cu at (164.8, 64.0)
- added kibuzzard-6A6CF79F: G***, kibuzzard-6A6CF79F, B.Cu at (164.6, 81.7)
- moved J16 4.89 mm to (150.8, 118.4), turned to 0 degrees
- moved H3 0.94 mm to (169.8, 122.0)
- moved TP1 0.49 mm to (145.5, 61.3)
- moved H6 0.48 mm to (169.9, 63.3)
- moved H1 0.39 mm to (96.8, 122.0)
- moved H5 0.38 mm to (96.8, 63.3)
Routing:
- net GND: track 106.7 -> 147.5 mm, vias 27 -> 37
- net /5V_P: track 160.3 -> 180.9 mm, vias 5 -> 7
- net /C7: track 54.6 -> 72.9 mm
- net /C6: track 41.8 -> 60.0 mm
- net /5V_P_USB: track 84.7 -> 81.0 mm, vias 3 -> 2
- net /15: track 45.8 -> 42.5 mm
- net /BAT: track 45.6 -> 48.5 mm
- net /39: track 115.2 -> 112.5 mm
- net /3V3: track 244.9 -> 242.4 mm
- net /VIN: track 25.3 -> 26.8 mm
- net /12V: track 122.6 -> 123.9 mm
- net /32: track 102.5 -> 101.5 mm
- net /R8: track 42.2 -> 41.4 mm
- net /33: track 51.8 -> 52.6 mm
- net /25: track 91.8 -> 92.5 mm
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Other:
- board text added: "- Omkar Nanajkar"
- board text added: "Put that back!"
- board text added: "sravjti.in"
