File: _restore_backup_2026-07-08T20-58-42-643/sra_board.kicad_pcb (KiCad board)
At the start: 2 copper layers, 97.6 x 65.8 mm, 165 parts, among them J10 Conn_01x03_Pin, J11 Conn_01x08_Pin, J12 Conn_01x07_Pin, J13 Conn_01x04_Pin, J14 Conn_01x02_Pin, J15 Conn_01x02_Pin, J16 Conn_01x02_Pin, J17 USB_C_Receptacle_USB2.0_16P, J18 Conn_01x10_Pin, J19 Conn_01x10_Pin, J20 Conn_01x10_Pin, J3 Conn_01x03_Pin, J5 Conn_01x03_Pin, J6 Conn_01x03_Pin, J7 Conn_01x03_Pin, J8 Conn_01x03_Pin, J9 Conn_01x03_Pin, Q1 SS8050, Q2 SS8050, Q3 AO4435, Q4 AO4468, SW3 SW_IO0, SW4 Switch, SW5 SW_EN, SW6 Switch, U2 ESP32-WROOM-32E, U4 ME6211C33M5, U5 CH340C, U6 TPS562202, U8 TB6612FNG H-bridge Motor Driv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

Commit message: Changed footprints of mounting holes, SMD fuses
Parts:
- removed U8: TB6612FNG H-bridge Motor Driver, Motor_driver:MODULE_ROB-14450
- J13: footprint Connector_PinSocket_2.54mm:PinSocket_1x04_P2.54mm_Vertical -> Connector_PinHeader_2.54mm:PinHeader_1x04_P2.54mm_Vertical
- J14, J15: footprint Connector_JST:JST_EH_S2B-EH_1x02_P2.50mm_Horizontal -> Connector_JST:JST_EH_B2B-EH-A_1x02_P2.50mm_Vertical
- moved J15 98.4 mm to (150.5, 100.9), turned to 0 degrees
- moved J14 92.4 mm to (150.5, 95.1), turned to 0 degrees
- moved J17 87.0 mm to (106.3, 205.4)
- moved TP1 77.3 mm to (109.9, 167.0)
- moved SW4 76.2 mm to (134.2, 150.6)
- moved SW6 76.2 mm to (134.2, 161.5)
- moved J10 64.0 mm to (162.3, 61.8), turned to 0 degrees
- moved J3 41.7 mm to (117.5, 101.5), turned to 0 degrees
- moved J6 34.2 mm to (124.4, 68.2), turned to 0 degrees
- moved J13 31.8 mm to (101.1, 116.3), turned to 0 degrees
- moved D66 29.2 mm to (139.6, 172.3)
- moved SW3 29.2 mm to (134.2, 172.1)
- moved U5 24.2 mm to (58.1, 183.0)
- moved J12 2.32 mm to (51.4, 57.7)
- moved J20 0.10 mm to (82.6, 81.9)
Other:
- board outline removed
