File: _restore_backup_2026-07-08T20-58-42-643/sra_board.kicad_sch (KiCad schematic)
At the start: 168 parts, among them J10 Conn_01x03_Pin, J11 Conn_01x08_Pin, J12 Conn_01x07_Pin, J13 Conn_01x04_Pin, J14 Conn_01x02_Pin, J15 Conn_01x02_Pin, J16 Conn_01x02_Pin, J17 USB_C_Receptacle_USB2.0_16P, J18 Conn_01x10_Pin, J19 Conn_01x10_Pin, J20 Conn_01x10_Pin, J3 Conn_01x03_Pin, J5 Conn_01x03_Pin, J6 Conn_01x03_Pin, J7 Conn_01x03_Pin, J8 Conn_01x03_Pin, J9 Conn_01x03_Pin, Q1 SS8050, Q2 SS8050, Q3 AO4435, Q4 AO4468, SW3 SW_IO0, SW4 Switch, SW5 SW_EN, SW6 Switch, U1 MAX7219CWG_T, U2 ESP32-WROOM-32E, U4 ME6211C33M5, U5 CH340C, U6 TPS562202, U7 CN3303, U8 TB6612FNG H-bridge Motor Driv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

Commit message: Changed footprints of mounting holes, SMD fuses
Parts:
- F1, F2: footprint Fuse:Fuse_1812_4532Metric -> Fuse:Fuse_Littelfuse-LVR100
- H1, H2, H3, H4, H5, H6: footprint MountingHole:MountingHole_3.2mm_M3_Pad_Via -> MountingHole:MountingHole_3.2mm_M3
- J13: footprint Connector_PinSocket_2.54mm:PinSocket_1x04_P2.54mm_Vertical -> Connector_PinHeader_2.54mm:PinHeader_1x04_P2.54mm_Vertical
- J14, J15: footprint Connector_JST:JST_EH_S2B-EH_1x02_P2.50mm_Horizontal -> Connector_JST:JST_EH_B2B-EH-A_1x02_P2.50mm_Vertical
- J16: footprint Connector_JST:JST_VH_B2PS-VH_1x02_P3.96mm_Horizontal -> Connector_JST:JST_EH_S2B-EH_1x02_P2.50mm_Horizontal
- U8: footprint Motor_driver:MODULE_ROB-14450 -> footprints:MODULE_ROB-14450
Changed lines of the file:
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@@
 			)
 		)
-		(property "Footprint" "MountingHole:MountingHole_3.2mm_M3_Pad_Via"
+		(property "Footprint" "MountingHole:MountingHole_3.2mm_M3"
 			(at 367.03 118.872 0)
 			(hide yes)
@@
 			)
 		)
-		(property "Footprint" "Connector_JST:JST_EH_S2B-EH_1x02_P2.50mm_Horizontal"
+		(property "Footprint" "Connector_JST:JST_EH_B2B-EH-A_1x02_P2.50mm_Vertical"
 			(at 112.776 131.572 0)
 			(hide yes)
@@
 			)
 		)
-		(property "Footprint" "Fuse:Fuse_1812_4532Metric"
+		(property "Footprint" "Fuse:Fuse_Littelfuse-LVR100"
 			(at 334.264 128.27 90)
 			(hide yes)
@@
 			)
 		)
-		(property "Footprint" "Motor_driver:MODULE_ROB-14450"
+		(property "Footprint" "footprints:MODULE_ROB-14450"
 			(at 170.434 35.56 0)
 			(hide yes)
@@
 			)
 		)
-		(property "Footprint" "MountingHole:MountingHole_3.2mm_M3_Pad_Via"
+		(property "Footprint" "MountingHole:MountingHole_3.2mm_M3"
 			(at 367.284 126.746 0)
 			(hide yes)
@@
 			)
 		)
-		(property "Footprint" "Connector_JST:JST_VH_B2PS-VH_1x02_P3.96mm_Horizontal"
+		(property "Footprint" "Connector_JST:JST_EH_S2B-EH_1x02_P2.50mm_Horizontal"
 			(at 260.858 127.254 0)
 			(hide yes)
@@
 			)
 		)
-		(property "Footprint" "MountingHole:MountingHole_3.2mm_M3_Pad_Via"
+		(property "Footprint" "MountingHole:MountingHole_3.2mm_M3"
 			(at 367.538 134.366 0)
 			(hide yes)
@@
 			)
 		)
-		(property "Footprint" "MountingHole:MountingHole_3.2mm_M3_Pad_Via"
+		(property "Footprint" "MountingHole:MountingHole_3.2mm_M3"
 			(at 388.112 118.872 0)
 			(hide yes)
@@
 			)
 		)
-		(property "Footprint" "Connector_JST:JST_EH_S2B-EH_1x02_P2.50mm_Horizontal"
+		(property "Footprint" "Connector_JST:JST_EH_B2B-EH-A_1x02_P2.50mm_Vertical"
 			(at 112.014 117.602 0)
 			(hide yes)
@@
 			)
 		)
-		(property "Footprint" "MountingHole:MountingHole_3.2mm_M3_Pad_Via"
+		(property "Footprint" "MountingHole:MountingHole_3.2mm_M3"
 			(at 388.874 134.62 0)
 			(hide yes)
@@
 			)
 		)
-		(property "Footprint" "Fuse:Fuse_1812_4532Metric"
+		(property "Footprint" "Fuse:Fuse_Littelfuse-LVR100"
 			(at 295.3004 127.4826 90)
 			(hide yes)
@@
 			)
 		)
-		(property "Footprint" "Connector_PinSocket_2.54mm:PinSocket_1x04_P2.54mm_Vertical"
+		(property "Footprint" "Connector_PinHeader_2.54mm:PinHeader_1x04_P2.54mm_Vertical"
 			(at 81.534 119.634 0)
 			(hide yes)
@@
 			)
 		)
-		(property "Footprint" "MountingHole:MountingHole_3.2mm_M3_Pad_Via"
+		(property "Footprint" "MountingHole:MountingHole_3.2mm_M3"
 			(at 388.62 126.492 0)
 			(hide yes)
