File: lsa/lsa.kicad_sch (KiCad schematic)
At the start: 16 parts, among them J2 Conn_01x08_Pin, U1 TCRT5000, U2 TCRT5000, U3 TCRT5000, U4 TCRT5000, U5 TCRT5000

Commit message: Switching to 10 pin FFC cable on both board and LSA, modifying silkscreen and holes for MPU
Parts:
- J2: value Conn_01x08_Pin -> Conn_01x10_Pin; footprint (none) -> Connector_FFC-FPC:JUSHUO_AFA07-S10FCA-00_1x10-1MP_P1.0mm_Horizontal; symbol Connector:Conn_01x08_Pin -> Connector:Conn_01x10_Pin
Connections:
- net +3V3: now also J2.10 (Pin_10), J2.7 (Pin_7), J2.8 (Pin_8), J2.9 (Pin_9); no longer J2.1 (Pin_1), J2.2 (Pin_2)
- net A0_36: now also J2.5 (Pin_5); no longer J2.4 (Pin_4)
- net A1_39: now also J2.4 (Pin_4); no longer J2.5 (Pin_5)
- net A2_34: now also J2.3 (Pin_3); no longer J2.6 (Pin_6)
- net A3_35: now also J2.2 (Pin_2); no longer J2.7 (Pin_7)
- net A4_32: now also J2.1 (Pin_1); no longer J2.8 (Pin_8)
- net GND: now also J2.6 (Pin_6); no longer J2.3 (Pin_3)
Changed lines of the file:
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@@
+	)
+	(junction
+		(at 264.668 60.96)
+		(diameter 0)
+		(color 0 0 0 0)
 	)
 	(junction
@@
 	)
 	(junction
+		(at 264.668 58.42)
+		(diameter 0)
+		(color 0 0 0 0)
+	)
+	(junction
 		(at 67.31 36.83)
 		(diameter 0)
@@
 		)
 	)
+	(wire
+		(pts
+			(xy 264.668 55.88) (xy 264.668 58.42)
+		)
+		(stroke
+			(width 0)
+			(type default)
+		)
+	)
 	(polyline
 		(pts
@@
 	(wire
 		(pts
+			(xy 262.89 63.5) (xy 264.668 63.5)
+		)
+		(stroke
+			(width 0)
+			(type default)
+		)
+	)
+	(wire
+		(pts
 			(xy 262.89 50.8) (xy 266.7 50.8)
 		)
@@
 		)
 	)
+	(wire
+		(pts
+			(xy 264.668 60.96) (xy 262.89 60.96)
+		)
+		(stroke
+			(width 0)
+			(type default)
+		)
+	)
 	(polyline
 		(pts
@@
 	(wire
 		(pts
+			(xy 264.668 63.5) (xy 264.668 60.96)
+		)
+		(stroke
+			(width 0)
+			(type default)
+		)
+	)
+	(wire
+		(pts
+			(xy 264.668 58.42) (xy 264.668 60.96)
+		)
+		(stroke
+			(width 0)
+			(type default)
+		)
+	)
+	(wire
+		(pts
 			(xy 262.89 53.34) (xy 266.7 53.34)
 		)
@@
 		(pts
 			(xy 153.67 36.83) (xy 153.67 38.1)
-		)
-		(stroke
-			(width 0)
-			(type default)
-		)
-	)
-	(wire
-		(pts
-			(xy 264.668 58.42) (xy 264.668 55.88)
 		)
 		(stroke
@@
 	)
 	(symbol
-		(lib_id "Connector:Conn_01x08_Pin")
+		(lib_id "Connector:Conn_01x10_Pin")
 		(at 257.81 50.8 0)
-		(mirror x)
 		(unit 1)
 		(body_style 1)
@@
 		(dnp no)
 		(property "Reference" "J2"
-			(at 258.445 63.5 0)
-			(show_name no)
-			(do_not_autoplace no)
-			(effects
-				(font
-					(size 1.27 1.27)
-				)
-			)
-		)
-		(property "Value" "Conn_01x08_Pin"
-			(at 258.445 60.96 0)
-			(show_name no)
-			(do_not_autoplace no)
-			(effects
-				(font
-					(size 1.27 1.27)
-				)
-			)
-		)
-		(property "Footprint" ""
+			(at 258.445 38.1 0)
+			(show_name no)
+			(do_not_autoplace no)
+			(effects
+				(font
+					(size 1.27 1.27)
+				)
+			)
+		)
+		(property "Value" "Conn_01x10_Pin"
+			(at 258.445 40.64 0)
+			(show_name no)
+			(do_not_autoplace no)
+			(effects
+				(font
+					(size 1.27 1.27)
+				)
+			)
+		)
+		(property "Footprint" "Connector_FFC-FPC:JUSHUO_AFA07-S10FCA-00_1x10-1MP_P1.0mm_Horizontal"
 			(at 257.81 50.8 0)
 			(hide yes)
@@
 			)
 		)
-		(property "Description" "Generic connector, single row, 01x08, script generated"
+		(property "Description" "Generic connector, single row, 01x10, script generated"
 			(at 257.81 50.8 0)
 			(hide yes)
@@
 		(pin "6"
 		)
+		(pin "9"
+		)
+		(pin "10"
+		)
 		(instances
